File: hardware/hfsdr.kicad_sch (KiCad schematic)
At the start: 3 parts, among them U1 SN74CBT3253, U2 XLV320ADC6120IRTER, Y1 Si5351A-B-GT

Commit message: Firmware
Parts:
- added J1: USB_C_Receptacle_USB2.0_16P, Connector_USB:USB_C_Receptacle_GCT_USB4105-xx-A_16P_TopMnt_Horizontal, symbol Connector:USB_C_Receptacle_USB2.0_16P
- added R1, R2: 5.1k, Resistor_SMD:R_0603_1608Metric_Pad0.98x0.95mm_HandSolder, symbol Device:R
- added U3: CH32V30xFxPx, Package_SO:TSSOP-20_4.4x6.5mm_P0.65mm, symbol MCU_WCH_CH32V3:CH32V30xFxPx
- added U4: XC6206PxxxMR, Package_TO_SOT_SMD:SOT-23-3, symbol Regulator_Linear:XC6206PxxxMR
- U1: footprint (none) -> Package_SO:TSSOP-16_4.4x5mm_P0.65mm
Connections:
- net MCU_XI: now reaches Y1.3 (XB)
- net MCU_XI: now also U3.19 (OSC_IN)
- net SCL: now reaches Y1.4 (SCL)
- net SCL: now also U2.13 (SCL), U3.3 (PB10)
- net SDA: now reaches Y1.5 (SDA)
- net SDA: now also U2.12 (SDA), U3.4 (PB11)
- net GND: now reaches Y1.8 (GND)
- net GND: now also U1.8 (GND), U2.10 (VSS), U2.15 (VSS), U2.20 (VSS), U2.21 (Thermal_Pad(VSS)), U2.5 (VSS), J1.A1 (GND), J1.A12 (GND), J1.B1 (GND), J1.B12 (GND), R1.1, R2.1, U3.18 (VSS), U4.1 (GND)
- net at U1.10 (2B1): now also U2.1 (IN1P)
- net at U1.11 (2B2): now also U2.3 (IN2P_GPI1)
- net at U1.12 (2B3): now also U2.4 (IN2M_GPO1)
- net at U1.13 (2B4): now also U2.2 (IN1M)
- net at U1.3 (1B4): no longer U2.2 (IN1M)
- net at U1.4 (1B3): no longer U2.4 (IN2M_GPO1)
- net at U1.5 (1B2): no longer U2.3 (IN2P_GPI1)
- net at U1.6 (1B1): no longer U2.1 (IN1P)
- net MCK: now reaches U2.11 (GPIO1)
- net MCK: now also U3.9 (PC6)
- net SD: now reaches U2.6 (SDOUT)
- net SD: now also U3.8 (PB15)
- net CK: now reaches U2.7 (BCLK)
- net CK: now also U3.6 (PB13)
- net WS: now reaches U2.8 (FSYNC)
- net WS: now also U3.5 (PB12)
- new net: J1.B5 (CC2), R1.2
- new net: J1.A5 (CC1), R2.2
- new net: J1.A4 (VBUS), J1.A9 (VBUS), J1.B4 (VBUS), J1.B9 (VBUS)
- new net: J1.A6 (D+), J1.B6 (D+), U3.17 (PB7)
- new net: J1.A7 (D-), J1.B7 (D-), U3.16 (PB6)
Other:
- moved on the sheet: U1, U2, Y1

Commit message: Update schematic
Parts:
- removed U1: SN74CBT3253, Package_SO:TSSOP-16_4.4x5mm_P0.65mm, symbol Analog_Switch:SN74CBT3253
- removed U2: XLV320ADC6120IRTER, RTE0020A-MFG, symbol 2025-06-21_15-05-27:XLV320ADC6120IRTER
- removed U3: CH32V30xFxPx, Package_SO:TSSOP-20_4.4x6.5mm_P0.65mm, symbol MCU_WCH_CH32V3:CH32V30xFxPx
- removed U4: XC6206PxxxMR, Package_TO_SOT_SMD:SOT-23-3, symbol Regulator_Linear:XC6206PxxxMR
- removed Y1: Si5351A-B-GT, Package_SO:MSOP-10_3x3mm_P0.5mm, symbol Oscillator:Si5351A-B-GT
- added C1, C10, C13, C14, C15, C16, C9: 1uF, Capacitor_SMD:C_0805_2012Metric_Pad1.18x1.45mm_HandSolder, symbol Device:C
- added C11, C12, C19, C2, C20, C4, C5, C6, C7, C8: 100nF, Capacitor_SMD:C_0805_2012Metric_Pad1.18x1.45mm_HandSolder, symbol Device:C
- added C3: 1nF, Capacitor_SMD:C_0805_2012Metric_Pad1.18x1.45mm_HandSolder, symbol Device:C
- added FB1: GZ2012D601TF, Inductor_SMD:L_0805_2012Metric_Pad1.05x1.20mm_HandSolder, symbol Device:FerriteBead_Small
- added R3, R4: 10k, Resistor_SMD:R_0603_1608Metric_Pad0.98x0.95mm_HandSolder, symbol Device:R
- added SW1: RST, Button_Switch_SMD:SW_Push_1P1T_XKB_TS-1187A, symbol Switch:SW_SPST
- added SW2: BOOT0, Button_Switch_SMD:SW_Push_1P1T_XKB_TS-1187A, symbol Switch:SW_SPST
- added U3: CH32V30xRxTx, Package_QFP:LQFP-64_10x10mm_P0.5mm, symbol MCU_WCH_CH32V3:CH32V30xRxTx
- added U4, U5: MD57E33QA3, Package_TO_SOT_SMD:SOT-23, symbol Regulator_Linear:TPS7A0520PDBZ
Connections:
- net CK: now also U3.34 (PB13)
- net GND: now also R1.2, C1.2, C10.2, C11.2, C13.2, C14.2, C15.2, C16.2, C19.2, C2.2, C20.1, C3.2, C4.2, C5.2, C6.2, C7.2, C8.2, C9.2, U3.12 (VSSA), U3.18 (VSS), U3.31 (VSS), U3.47 (VSS), U3.63 (VSS), U4.1 (GND), U5.1 (GND); no longer R1.1
- net MCK: now also U3.37 (PC6)
- net MCU_XI: now also C12.2
- net SCL: now also U3.29 (PB10)
- net SD: now also U3.36 (PB15)
- net SDA: now also U3.30 (PB11)
- net WS: now also U3.33 (PB12)
- net at J1.B5 (CC2): now also R1.1; no longer R1.2
- net +5V: now reaches J1.A4 (VBUS), J1.A9 (VBUS), J1.B4 (VBUS), J1.B9 (VBUS)
- net +5V: now also C1.1, C13.1, C16.1, C2.1, C3.1, U4.2 (VO), U5.2 (VO)
- net DP: now reaches J1.A6 (D+), J1.B6 (D+)
- net DP: now also U3.59 (PB7)
- net DM: now reaches J1.A7 (D-), J1.B7 (D-)
- net DM: now also U3.58 (PB6)
- new net: R4.2, U3.7 (~{RST})
- new net: C12.1, U3.5 (OSC_IN)
- new net: C19.1, R3.2, SW2.2 (B)
- new net: C11.1, FB1.2, U3.13 (VDDA)
- new net: R3.1, U3.60 (BOOT0)
- new net: C20.2, SW1.1 (A)
- new net +3.3V: C10.1, C14.1, C4.1, C5.1, C6.1, C7.1, C8.1, C9.1, FB1.1, R4.1, SW1.2 (B), SW2.1 (A), U3.1 (VBAT), U3.19 (VDD), U3.32 (VIO), U3.48 (VDD), U3.64 (VIO), U4.3 (VI)
- new net +3.3VA: C15.1, U5.3 (VI)
Other:
- added sheet RF (rf.kicad_sch)
- moved on the sheet: J1, R1, R2

Commit message: amp and audio
Parts:
- removed C13, C14, C15, C16: 1uF, Capacitor_SMD:C_0805_2012Metric_Pad1.18x1.45mm_HandSolder, symbol Device:C
- removed U4, U5: MD57E33QA3, Package_TO_SOT_SMD:SOT-23, symbol Regulator_Linear:TPS7A0520PDBZ
- added C24: 100nF, Capacitor_SMD:C_0805_2012Metric_Pad1.18x1.45mm_HandSolder, symbol Device:C
- added C25: 1uF, Capacitor_SMD:C_0805_2012Metric_Pad1.18x1.45mm_HandSolder, symbol Device:C
- added FB4, FB5: GZ2012D601TF, Inductor_SMD:L_0805_2012Metric_Pad1.05x1.20mm_HandSolder, symbol Device:FerriteBead_Small
- added U8: NS4165B, easyeda:ESOP-8_L4.9-W3.9-P1.27-LS6.0-BL-EP, symbol easyeda:NS4165B
Connections:
- net +3.3V: now also U8.6 (VDD)
- net +5V: no longer C1.1, C2.1, C3.1, J1.A4 (VBUS), J1.A9 (VBUS), J1.B4 (VBUS), J1.B9 (VBUS)
- net GND: now also C25.1, U8.7 (GND)
- net DAC1_OUT: now reaches U3.20 (PA4)
- net DAC1_OUT: now also C24.1
- net DAC2_OUT: now reaches U3.21 (PA5)
- new net: C24.2, U8.4 (INN)
- new net: FB4.1, U8.8 (VOP)
- new net: C25.2, U8.2 (Bypass)
- new net: FB5.2, U8.5 (VON)
- new net VBUS: C1.1, C2.1, C3.1, J1.A4 (VBUS), J1.A9 (VBUS), J1.B4 (VBUS), J1.B9 (VBUS)
Other:
- added sheet Power (power.kicad_sch)
- moved on the sheet: C1, C2, C3, J1, R1, R2

Commit message: arrange pcb
Parts:
- removed C24: 100nF, Capacitor_SMD:C_0805_2012Metric_Pad1.18x1.45mm_HandSolder, symbol Device:C
- removed C25: 1uF, Capacitor_SMD:C_0805_2012Metric_Pad1.18x1.45mm_HandSolder, symbol Device:C
- removed FB4, FB5: GZ2012D601TF, Inductor_SMD:L_0805_2012Metric_Pad1.05x1.20mm_HandSolder, symbol Device:FerriteBead_Small
- removed U8: NS4165B, easyeda:ESOP-8_L4.9-W3.9-P1.27-LS6.0-BL-EP, symbol easyeda:NS4165B
- R1, R2, R3, R4: footprint Resistor_SMD:R_0603_1608Metric_Pad0.98x0.95mm_HandSolder -> Resistor_SMD:R_0805_2012Metric_Pad1.20x1.40mm_HandSolder
Other:
- added sheet Audio (audio.kicad_sch)

Commit message: battery switching
Parts:
- U3: symbol MCU_WCH_CH32V3:CH32V30xRxTx -> MCU_WCH_RiscV:CH32V30xRxTx
Changed lines of the file:
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@@
 	)
 	(symbol
-		(lib_id "MCU_WCH_CH32V3:CH32V30xRxTx")
+		(lib_id "MCU_WCH_RiscV:CH32V30xRxTx")
 		(at 142.24 93.98 0)
 		(unit 1)
@@
 					(unit 1)
 				)
-			)
-		)
-	)
-	(symbol
-		(lib_id "power:+5V")
-		(at 195.58 17.78 0)
-		(unit 1)
-		(exclude_from_sim no)
-		(in_bom yes)
-		(on_board yes)
-		(dnp no)
-		(fields_autoplaced yes)
-		(property "Reference" "#PWR08"
-			(at 195.58 21.59 0)
-			(effects
-				(font
-					(size 1.27 1.27)
-				)
-				(hide yes)
-			)
-		)
-		(property "Value" "+5V"
-			(at 195.58 12.7 0)
-			(effects
-				(font
-					(size 1.27 1.27)
-				)
-			)
-		)
-		(property "Footprint" ""
-			(at 195.58 17.78 0)
-			(effects
-				(font
-					(size 1.27 1.27)
-				)
-				(hide yes)
-			)
-		)
-		(property "Datasheet" ""
-			(at 195.58 17.78 0)
-			(effects
-				(font
-					(size 1.27 1.27)
-				)
-				(hide yes)
-			)
-		)
-		(property "Description" "Power symbol creates a global label with name \"+5V\""
-			(at 195.58 17.78 0)
-			(effects
-				(font
-					(size 1.27 1.27)
-				)
-				(hide yes)
-			)
-		)
-		(pin "1"
-		)
-		(instances
-			(project "hfsdr"
-				(path "/a11445ed-c3bd-4d1c-a039-1c09b0dceab8"
-					(reference "#PWR08")
-					(unit 1)
-				)

Commit message: initial component layout
Parts:
- C3: value 1nF -> 2.2nF
Changed lines of the file:
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@@
 			)
 		)
-		(property "Value" "1nF"
+		(property "Value" "2.2nF"
 			(at 212.09 24.1299 0)
 			(effects

Commit message: initial screen
Parts:
- added FPC1: FPC-05F-18PH20, easyeda:FPC-SMD_18P-P0.50_FPC-05F-18PH20, symbol easyeda:FPC-05F-18PH20
Connections:
- net +3.3V: now also FPC1.3, FPC1.4
- net GND: now also FPC1.1, FPC1.12, FPC1.18, FPC1.5, FPC1.6
- net SCL_SCK: now reaches U3.55 (PB3)
- net SCL_SCK: now also FPC1.9
- net SDA_MOSI: now reaches U3.57 (PB5)
- net SDA_MOSI: now also FPC1.10
- new net CS: FPC1.8
- new net RS: FPC1.7
- new net RST: FPC1.11

Commit message: feat: add rough art
Parts:
- added H1: MountingHole_Pad, MountingHole:MountingHole_3.2mm_M3_Pad, symbol Mechanical:MountingHole_Pad
Changed lines of the file:
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@@
+	)
+	(symbol
+		(lib_id "Mechanical:MountingHole_Pad")
+		(at 222.25 76.2 0)
+		(unit 1)
+		(exclude_from_sim yes)
+		(in_bom no)
+		(on_board yes)
+		(dnp no)
+		(fields_autoplaced yes)
+		(property "Reference" "H1"
+			(at 224.79 73.6599 0)
+			(effects
+				(font
+					(size 1.27 1.27)
+				)
+				(justify left)
+			)
+		)
+		(property "Value" "MountingHole_Pad"
+			(at 224.79 76.1999 0)
+			(effects
+				(font
+					(size 1.27 1.27)
+				)
+				(justify left)
+			)
+		)
+		(property "Footprint" "MountingHole:MountingHole_3.2mm_M3_Pad"
+			(at 222.25 76.2 0)
+			(effects
+				(font
+					(size 1.27 1.27)
+				)
+				(hide yes)
+			)
+		)
+		(property "Datasheet" "~"
+			(at 222.25 76.2 0)
+			(effects
+				(font
+					(size 1.27 1.27)
+				)
+				(hide yes)
+			)
+		)
+		(property "Description" "Mounting Hole with connection"
+			(at 222.25 76.2 0)
+			(effects
+				(font
+					(size 1.27 1.27)
+				)
+				(hide yes)
+			)
+		)
+		(pin "1"
+		)
+		(instances
+			(project ""
+				(path "/a11445ed-c3bd-4d1c-a039-1c09b0dceab8"
+					(reference "H1")
+					(unit 1)
+				)
+			)
+		)
 	)
 	(symbol
