File: hardware/hfsdr.kicad_pcb (KiCad board)
At the start: 4 copper layers, 99.8 x 73.8 mm, 129 parts, among them J1 USB_C_Receptacle_USB2.0_16P, J2 AudioPlug4, J4 JST PH S2B, Q1 AO3401A, SW1 RST, SW2 BOOT0, SW3 MST-22D18G4-WT, SW4 RotaryEncoder_Switch, U1 SN74CBT3253, U2 XLV320ADC6120IRTER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

Commit message: feat: added silkscreen labels
Other:
- board text added: "ADC"
- board text added: "Amplifier"
- board text added: "Clock"
- board text added: "MCU"
- board text added: "Quad Demux"
- board text added: "RF RX"
- board text added: "USB Data + Power"
- board text removed: "RX Chain"
Changed lines of the file:
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@@
 		(tags "capacitor handsolder")
 		(property "Reference" "C48"
-			(at -2.692886 -0.904372 90)
+			(at -0.017549 -0.147516 180)
 			(layer "F.SilkS")
 			(effects
@@
 		(tags "test point SMD pad rectangle square")
 		(property "Reference" "TP7"
-			(at 0 -1.448 0)
+			(at 0.0585 2.028071 0)
 			(layer "F.SilkS")
 			(effects
@@
 		(tags "capacitor handsolder")
 		(property "Reference" "C12"
-			(at -0.045131 1.859804 0)
+			(at -0.261252 0.034734 0)
 			(layer "F.SilkS")
 			(effects
@@
 		(layer "F.SilkS")
 	)
+	(gr_arc
+		(start 141.53791 56.428515)
+		(mid 140.501923 57.411102)
+		(end 139.517101 56.377239)
+		(stroke
+			(width 0.1)
+			(type default)
+		)
+		(layer "F.SilkS")
+	)
 	(gr_line
 		(start 117.928227 47.837759)
@@
 		(layer "F.SilkS")
 	)
+	(gr_line
+		(start 129.940351 82.58634)
+		(end 131.398386 82.58634)
+		(stroke
+			(width 0.1)
+			(type default)
+		)
+		(layer "F.SilkS")
+	)
+	(gr_line
+		(start 134.632573 84.344819)
+		(end 136.382215 84.344819)
+		(stroke
+			(width 0.1)
+			(type default)
+		)
+		(layer "F.SilkS")
+	)
 	(gr_circle
 		(center 120.00712 49.916652)
@@
 		(layer "F.SilkS")
 	)
+	(gr_line
+		(start 131.398386 84.335983)
+		(end 131.398386 82.58634)
+		(stroke
+			(width 0.1)
+			(type default)
+		)
+		(layer "F.SilkS")
+	)
 	(gr_circle
 		(center 89.895936 64.812143)
@@
 	)
 	(gr_line
+		(start 131.398386 84.335983)
+		(end 133.148028 84.335983)
+		(stroke
+			(width 0.1)
+			(type default)
+		)
+		(layer "F.SilkS")
+	)
+	(gr_line
+		(start 134.632573 84.344819)
+		(end 134.632573 82.595176)
+		(stroke
+			(width 0.1)
+			(type default)
+		)
+		(layer "F.SilkS")
+	)
+	(gr_line
 		(start 90.641819 60.611773)
 		(end 93.97138 60.611773)
@@
 		(layer "F.SilkS")
 	)
+	(gr_line
+		(start 133.183374 84.318308)
+		(end 133.183374 82.568665)
+		(stroke
+			(width 0.1)
+			(type default)
+		)
+		(layer "F.SilkS")
+	)
 	(gr_arc
 		(start 156.288506 46.845201)
@@
 		(layer "F.SilkS")
 	)
+	(gr_line
+		(start 133.174538 82.595176)
+		(end 134.632573 82.595176)
+		(stroke
+			(width 0.1)
+			(type default)
+		)
+		(layer "F.SilkS")
+	)
 	(gr_rect
 		(start 84.219278 72.456499)
@@
 		(layer "F.SilkS")
 	)
+	(gr_line
+		(start 129.949187 84.309472)
+		(end 129.949187 82.559829)
+		(stroke
+			(width 0.1)
+			(type default)
+		)
+		(layer "F.SilkS")
+	)
 	(gr_arc
 		(start 156.343423 45.673625)
@@
 		(layer "F.SilkS")
 	)
+	(gr_arc
+		(start 137.496292 56.325963)
+		(mid 138.532279 55.343376)
+		(end 139.517101 56.377239)
+		(stroke
+			(width 0.1)
+			(type default)
+		)
+		(layer "F.SilkS")
+	)
 	(gr_rect
 		(start 63.316265 35.202685)
@@
 		)
 	)
+	(gr_text "Clock"
+		(at 130.072731 81.668626 0)
+		(layer "F.SilkS" knockout)
+		(effects
+			(font
+				(size 1 1)
+				(thickness 0.2)
+				(bold yes)
+			)
+			(justify left bottom)
+		)
+	)
+	(gr_text "Quad Demux"
+		(at 156.162657 68.950789 90)
+		(layer "F.SilkS" knockout)
+		(effects
+			(font
+				(size 1 1)
+				(thickness 0.2)
+				(bold yes)
+			)
+			(justify left bottom)
+		)
+	)
 	(gr_text "ON"
 		(at 85.147654 104.450627 0)
@@
 		)
 	)
-	(gr_text "RX\nChain"
-		(at 155.066911 54.707374 0)
+	(gr_text "USB Data + Power"
+		(at 68.291526 104.88259 0)
+		(layer "F.SilkS" knockout)
+		(effects
+			(font
+				(size 1 1)
+				(thickness 0.2)
+				(bold yes)
+			)
+			(justify left bottom)
+		)
+	)
+	(gr_text "MCU"
+		(at 109.014803 60.00595 0)
+		(layer "F.SilkS" knockout)
+		(effects
+			(font
+				(size 1 1)
+				(thickness 0.2)
+				(bold yes)
+			)
+			(justify left bottom)
+		)
+	)
+	(gr_text "ADC"
+		(at 137.400848 59.600012 0)
+		(layer "F.SilkS" knockout)
+		(effects
+			(font
+				(size 1 1)
+				(thickness 0.2)
+				(bold yes)
+			)
+			(justify left bottom)
+		)
+	)
+	(gr_text "Amplifier"
+		(at 154.542249 52.567775 0)
 		(layer "F.SilkS" knockout)
 		(effects
@@
 		(layer "F.SilkS" knockout)
 		(effects
+			(font
+				(size 1 1)
+				(thickness 0.2)
+				(bold yes)
+			)
+			(justify left bottom)
+		)
+	)
+	(gr_text "RF RX"
+		(at 152.391164 44.275338 0)
+		(layer "F.SilkS" knockout)
+		(effects

Commit message: Ready for production
Parts:
- added C53: 1uF, Capacitor_SMD:C_0805_2012Metric_Pad1.18x1.45mm_HandSolder, F.Cu at (80.5, 100.5)
- added C54: 100nF, Capacitor_SMD:C_0805_2012Metric_Pad1.18x1.45mm_HandSolder, F.Cu at (80.5, 102.5)
- C24, C26: value 470nF -> 1uF
- C3, C43, C44, C45, C46: value 2.2nF -> 10nF
- R15, R16: value 4.7k -> 2k
Routing:
- net VBUS: track 63.5 -> 67.7 mm

Commit message: production
Parts:
- added D5: BAV99, Package_TO_SOT_SMD:SOT-23, F.Cu at (144.1, 47.3)
- added JP2: Shield GND, Jumper:SolderJumper-2_P1.3mm_Open_RoundedPad1.0x1.5mm, F.Cu at (65.8, 89.3)
- U1: value SN74CBT3253 -> SN74CBTLV3253
Connections:
- SW4 pad MP: (no net) -> GND
- U8 pad 5: unconnected-(U8-~{SD}-Pad5) -> PA11
Routing:
- net GND: track 173.8 -> 214.8 mm, vias 50 -> 65
- net DAC2_OUT: track 62.1 -> 34.4 mm
- net PA11: track 16.1 -> 39.8 mm
- net +3.3V: track 107.6 -> 124.5 mm
- net Net-(C29-Pad2): track 5.97 -> 12.2 mm
- net unconnected-(J1-SHIELD-PadS1): track 0.00 -> 2.32 mm
- net DAC1_OUT: track 47.2 -> 46.0 mm

Commit message: unsaved stuff
Parts:
- added C55: 100nF, Capacitor_SMD:C_0805_2012Metric_Pad1.18x1.45mm_HandSolder, F.Cu at (139.4, 86.3)
- added C56: 1uF, Capacitor_SMD:C_0805_2012Metric_Pad1.18x1.45mm_HandSolder, F.Cu at (139.4, 88.3)
Routing:
- net +3.3V: track 124.5 -> 107.6 mm
- net +5V: track 78.3 -> 79.6 mm
- net GND: vias 65 -> 67
