File: hardware/audio.kicad_sch (KiCad schematic)
At the start: 12 parts, among them J2 AudioPlug4, U8 LM4809

Commit message: V3 changes
Parts:
- added C57, C58, C59, C60: 220pF, Capacitor_SMD:C_0805_2012Metric_Pad1.18x1.45mm_HandSolder, symbol Device:C
- added R23, R24: 10k, Resistor_SMD:R_0805_2012Metric_Pad1.20x1.40mm_HandSolder, symbol Device:R
- R5, R6: value 20k -> 10k
Connections:
- net GND: now also C59.2, C60.2
- net at C24.1: now also R24.2; no longer R6.2
- net at R5.1: now also C60.1, R23.2; no longer C26.1
- net at R10.1, R6.1, U8.6 (IN2): now also C57.2
- net at C31.1, R10.2, U8.7 (V02): now also C57.1
- net at C30.1, R11.2, U8.1 (V01): now also C58.1
- net at R11.1, R5.2, U8.2 (IN1): now also C58.2
- new net: C26.1, R23.1
- new net: C59.1, R24.1, R6.2
Other:
- moved on the sheet: C24, C26, R5, R6
